File: Hardware/v1.sch (EAGLE design)
At the start: 69 parts, among them CN1 629105150521, CN2 TSW-120-08-L-S-RA, CN3 1734354-1, CN4 1-1734530-1, IC1 ADUM3160BRWZ, IC2 TUSB2046BIRHBT, IC3 IC_MAX3313, IC4 FT2232D, IC6 PCM2903C

Commit message: complete apart from sound card and PIC
Parts:
- added C31: 1uF, rcl:C-EUC0402
- added C32: 100nF, rcl:C-EUC0402
- C25: value 100nF -> 1uF
- C30: value 1uF -> 100nF
- R8, R9: device rcl:R-EU_R0603 -> rcl:R-EU_R0402
Connections:
- net +5V: now also C31.1, C32.1
- net ACC_ALC: now also R8.1
- net ACC_BND0: now also RN1.1A; no longer RN1.3A
- net ACC_BND1: now also RN1.4A; no longer RN1.1A
- net ACC_BND2: now also RN1.3A; no longer RN1.2A
- net ACC_BND3: now also RN1.2A; no longer RN1.4A
- net GND: now also C31.2, C32.2
Other:
- moved on the sheet: C29, C30, R8
Changed lines of the file:
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@@
 <part name="FRAME6" library="frames" deviceset="A4L-LOC" device=""/>
 <part name="IC6" library="texas" deviceset="PCM290*" device="" technology="2E" value="PCM2903C"/>
-<part name="C25" library="rcl" deviceset="C-EU" device="C0402" value="100nF"/>
+<part name="C25" library="rcl" deviceset="C-EU" device="C0402" value="1uF"/>
 <part name="P+7" library="supply1" deviceset="+5V" device=""/>
 <part name="GND13" library="supply1" deviceset="GND" device=""/>
@@
 <part name="R29" library="rcl" deviceset="R-EU_" device="R0805" value="137k"/>
 <part name="L1" library="m0wut" deviceset="INDUCTOR" device="" value="100uH"/>
-<part name="C29" library="rcl" deviceset="C-EU" device="C0402" value="100nF"/>
-<part name="C30" library="rcl" deviceset="C-EU" device="C0402" value="1uF"/>
+<part name="C30" library="rcl" deviceset="C-EU" device="C0402" value="100nF"/>
 <part name="RN1" library="m0wut" deviceset="R_BOURNS_CAY16-J4" device="" value="2k2"/>
 <part name="P+8" library="supply1" deviceset="+5V" device=""/>
-<part name="R8" library="rcl" deviceset="R-EU_" device="R0603" value="69k8"/>
-<part name="R9" library="rcl" deviceset="R-EU_" device="R0603" value="100k"/>
+<part name="R8" library="rcl" deviceset="R-EU_" device="R0402" value="69k8"/>
+<part name="R9" library="rcl" deviceset="R-EU_" device="R0402" value="100k"/>
 <part name="GND19" library="supply1" deviceset="GND" device=""/>
 <part name="P+10" library="supply1" deviceset="+5V" device=""/>
+<part name="C31" library="rcl" deviceset="C-EU" device="C0402" value="1uF"/>
+<part name="C32" library="rcl" deviceset="C-EU" device="C0402" value="100nF"/>
+<part name="GND17" library="supply1" deviceset="GND" device=""/>
+<part name="C29" library="rcl" deviceset="C-EU" device="C0402" value="100nF"/>
 </parts>
 <sheets>
@@
 <instance part="VDD1" gate="G$1" x="147.32" y="149.86"/>
 <instance part="VDD2" gate="G$1" x="83.82" y="111.76"/>
-<instance part="C29" gate="G$1" x="231.14" y="106.68"/>
-<instance part="C30" gate="G$1" x="243.84" y="106.68"/>
+<instance part="C30" gate="G$1" x="231.14" y="106.68"/>
+<instance part="C29" gate="G$1" x="208.28" y="106.68"/>
 </instances>
 <busses>
@@
 <wire x1="218.44" y1="99.06" x2="218.44" y2="101.6" width="0.1524" layer="91"/>
 <pinref part="C30" gate="G$1" pin="2"/>
+<wire x1="231.14" y1="101.6" x2="218.44" y2="101.6" width="0.1524" layer="91"/>
+<junction x="218.44" y="101.6"/>
 <pinref part="C29" gate="G$1" pin="2"/>
-<wire x1="243.84" y1="101.6" x2="231.14" y2="101.6" width="0.1524" layer="91"/>
-<wire x1="231.14" y1="101.6" x2="218.44" y2="101.6" width="0.1524" layer="91"/>
-<junction x="231.14" y="101.6"/>
-<junction x="218.44" y="101.6"/>
+<wire x1="218.44" y1="101.6" x2="208.28" y2="101.6" width="0.1524" layer="91"/>
 </segment>
 <segment>
@@
 <pinref part="C25" gate="G$1" pin="1"/>
 <wire x1="218.44" y1="109.22" x2="218.44" y2="111.76" width="0.1524" layer="91"/>
-<pinref part="C29" gate="G$1" pin="1"/>
-<wire x1="231.14" y1="109.22" x2="218.44" y2="109.22" width="0.1524" layer="91"/>
 <junction x="218.44" y="109.22"/>
 <pinref part="C30" gate="G$1" pin="1"/>
-<wire x1="231.14" y1="109.22" x2="243.84" y2="109.22" width="0.1524" layer="91"/>
-<junction x="231.14" y="109.22"/>
+<wire x1="218.44" y1="109.22" x2="231.14" y2="109.22" width="0.1524" layer="91"/>
+<pinref part="C29" gate="G$1" pin="1"/>
+<wire x1="218.44" y1="109.22" x2="208.28" y2="109.22" width="0.1524" layer="91"/>
 </segment>
 <segment>
@@
 <instance part="RN1" gate="G$1" x="99.06" y="104.14" rot="MR270"/>
 <instance part="P+8" gate="1" x="96.52" y="127"/>
-<instance part="R8" gate="G$1" x="63.5" y="58.42" rot="R90"/>
+<instance part="R8" gate="G$1" x="63.5" y="60.96" rot="R90"/>
 <instance part="R9" gate="G$1" x="63.5" y="45.72" rot="R90"/>
 <instance part="GND19" gate="1" x="63.5" y="35.56"/>
-<instance part="P+10" gate="1" x="63.5" y="68.58"/>
+<instance part="P+10" gate="1" x="63.5" y="71.12"/>
+<instance part="C31" gate="G$1" x="109.22" y="116.84"/>
+<instance part="C32" gate="G$1" x="119.38" y="116.84"/>
+<instance part="GND17" gate="1" x="114.3" y="104.14"/>
 </instances>
 <busses>
@@
 <wire x1="63.5" y1="40.64" x2="63.5" y2="38.1" width="0.1524" layer="91"/>
 </segment>
+<segment>
+<pinref part="C31" gate="G$1" pin="2"/>
+<wire x1="109.22" y1="111.76" x2="109.22" y2="109.22" width="0.1524" layer="91"/>
+<pinref part="C32" gate="G$1" pin="2"/>
+<wire x1="109.22" y1="109.22" x2="114.3" y2="109.22" width="0.1524" layer="91"/>
+<wire x1="114.3" y1="109.22" x2="119.38" y2="109.22" width="0.1524" layer="91"/>
+<wire x1="119.38" y1="109.22" x2="119.38" y2="111.76" width="0.1524" layer="91"/>
+<pinref part="GND17" gate="1" pin="GND"/>
+<wire x1="114.3" y1="106.68" x2="114.3" y2="109.22" width="0.1524" layer="91"/>
+<junction x="114.3" y="109.22"/>
+</segment>
 </net>
 <net name="232_COM" class="0">
@@
 <segment>
 <pinref part="R27" gate="G$1" pin="1"/>
-<wire x1="104.14" y1="58.42" x2="99.06" y2="58.42" width="0.1524" layer="91"/>
 <label x="81.28" y="58.928" size="1.27" layer="95"/>
-<pinref part="RN1" gate="G$1" pin="3A"/>
-<wire x1="99.06" y1="58.42" x2="81.28" y2="58.42" width="0.1524" layer="91"/>
-<wire x1="99.06" y1="96.52" x2="99.06" y2="58.42" width="0.1524" layer="91"/>
-<junction x="99.06" y="58.42"/>
+<wire x1="104.14" y1="58.42" x2="93.98" y2="58.42" width="0.1524" layer="91"/>
+<pinref part="RN1" gate="G$1" pin="1A"/>
+<wire x1="93.98" y1="58.42" x2="81.28" y2="58.42" width="0.1524" layer="91"/>
+<wire x1="93.98" y1="96.52" x2="93.98" y2="58.42" width="0.1524" layer="91"/>
+<junction x="93.98" y="58.42"/>
 </segment>
 </net>
@@
 <segment>
 <pinref part="R28" gate="G$1" pin="1"/>
-<wire x1="104.14" y1="55.88" x2="101.6" y2="55.88" width="0.1524" layer="91"/>
 <label x="81.28" y="56.388" size="1.27" layer="95"/>
-<pinref part="RN1" gate="G$1" pin="4A"/>
-<wire x1="101.6" y1="55.88" x2="81.28" y2="55.88" width="0.1524" layer="91"/>
-<wire x1="101.6" y1="96.52" x2="101.6" y2="55.88" width="0.1524" layer="91"/>
-<junction x="101.6" y="55.88"/>
+<wire x1="104.14" y1="55.88" x2="96.52" y2="55.88" width="0.1524" layer="91"/>
+<pinref part="RN1" gate="G$1" pin="2A"/>
+<wire x1="96.52" y1="55.88" x2="81.28" y2="55.88" width="0.1524" layer="91"/>
+<wire x1="96.52" y1="96.52" x2="96.52" y2="55.88" width="0.1524" layer="91"/>
+<junction x="96.52" y="55.88"/>
 </segment>
 </net>
@@
 <segment>
 <pinref part="R24" gate="G$1" pin="1"/>
-<wire x1="104.14" y1="68.58" x2="96.52" y2="68.58" width="0.1524" layer="91"/>
 <label x="81.28" y="69.088" size="1.27" layer="95"/>
-<pinref part="RN1" gate="G$1" pin="2A"/>
-<wire x1="96.52" y1="68.58" x2="81.28" y2="68.58" width="0.1524" layer="91"/>
-<wire x1="96.52" y1="96.52" x2="96.52" y2="68.58" width="0.1524" layer="91"/>
-<junction x="96.52" y="68.58"/>
+<wire x1="104.14" y1="68.58" x2="99.06" y2="68.58" width="0.1524" layer="91"/>
+<pinref part="RN1" gate="G$1" pin="3A"/>
+<wire x1="99.06" y1="68.58" x2="81.28" y2="68.58" width="0.1524" layer="91"/>
+<wire x1="99.06" y1="96.52" x2="99.06" y2="68.58" width="0.1524" layer="91"/>
+<junction x="99.06" y="68.58"/>
 </segment>
 </net>
@@
 <wire x1="63.5" y1="53.34" x2="63.5" y2="50.8" width="0.1524" layer="91"/>
 <junction x="63.5" y="53.34"/>
+<pinref part="R8" gate="G$1" pin="1"/>
+<wire x1="63.5" y1="55.88" x2="63.5" y2="53.34" width="0.1524" layer="91"/>
 </segment>
 </net>
@@
 <segment>
 <pinref part="R19" gate="G$1" pin="1"/>
-<wire x1="104.14" y1="83.82" x2="93.98" y2="83.82" width="0.1524" layer="91"/>
 <label x="81.28" y="84.328" size="1.27" layer="95"/>
-<pinref part="RN1" gate="G$1" pin="1A"/>
-<wire x1="93.98" y1="83.82" x2="81.28" y2="83.82" width="0.1524" layer="91"/>
-<wire x1="93.98" y1="96.52" x2="93.98" y2="83.82" width="0.1524" layer="91"/>
-<junction x="93.98" y="83.82"/>
+<wire x1="104.14" y1="83.82" x2="101.6" y2="83.82" width="0.1524" layer="91"/>
+<pinref part="RN1" gate="G$1" pin="4A"/>
+<wire x1="101.6" y1="83.82" x2="81.28" y2="83.82" width="0.1524" layer="91"/>
+<wire x1="101.6" y1="96.52" x2="101.6" y2="83.82" width="0.1524" layer="91"/>
+<junction x="101.6" y="83.82"/>
 </segment>
 </net>
@@
 <pinref part="P+8" gate="1" pin="+5V"/>
 <wire x1="96.52" y1="124.46" x2="96.52" y2="119.38" width="0.1524" layer="91"/>
+<pinref part="C31" gate="G$1" pin="1"/>
+<wire x1="101.6" y1="119.38" x2="109.22" y2="119.38" width="0.1524" layer="91"/>
+<junction x="101.6" y="119.38"/>
+<pinref part="C32" gate="G$1" pin="1"/>
+<wire x1="109.22" y1="119.38" x2="119.38" y2="119.38" width="0.1524" layer="91"/>
+<junction x="109.22" y="119.38"/>
 </segment>
 <segment>
 <pinref part="R8" gate="G$1" pin="2"/>
 <pinref part="P+10" gate="1" pin="+5V"/>
-<wire x1="63.5" y1="63.5" x2="63.5" y2="66.04" width="0.1524" layer="91"/>
-</segment>
-</net>
+<wire x1="63.5" y1="68.58" x2="63.5" y2="66.04" width="0.1524" layer="91"/>
+</segment>
+</net>

Commit message: destruction in the name of progress...
Parts:
- removed C3, C4, C5: 100nF, rcl:C-EUC0603
- removed IC6: PCM2903C, texas:PCM2902E
- added C33, C34: 1nF, rcl:C-EUC0402
- added CAN1: SHIELDING_CAN, m0wut:SHIELDING_CAN
- added D2: BZT52C3V0-7-F, adafruit:DIODESOD-123
- added L2, L3, L4, L5, L6, L7: 100uH, m0wut:INDUCTOR
- added R12: 220, rcl:R-EU_R0402
- CN1: value 629105150521 -> 54819-0519; device m0wut:USBWURTH -> m0wut:USBMOLEX_MINI
- IC3: value IC_MAX3313 -> (none); device m0wut:IC_MAX3313 -> m0wut:IC_MAX3375
Connections:
- removed net 232_COM: CN2.P$1
- removed net N$8: C4.1, IC3.V-
- removed net RS232(K2_TO_PIC): IC3.RIN
- removed net RS232(PIC_TO_K3): IC3.TOUT
- removed net UART(K3_TO_PIC): IC3.ROUT
- removed net UART(PIC_TO_K3): IC3.TIN
- new net 3V3_HUB: C10.1, C11.1, C9.1, IC2.!EXTMEM, IC2.VCC, IC2.VCC@1, L6.2, R5.1
- new net N$18: C33.1, CN3.2, L2.2
- new net N$188: IC3.OH, L2.1
- new net N$189: D2.C, IC3.IH, R12.1
- new net N$19: C6.1, C7.1, IC1.PIN, IC1.SPD, IC1.VBUS2, IC1.VDD2, L5.1
- new net N$4: C34.1, CN3.3, L3.2
- new net USB_IN_GND: C1.2, C2.2, CN1.GND, D1.GND, IC1.GND1, IC1.GND1_2, L7.1
- net +3V3: now also L4.1, L5.2, L6.1; no longer C10.1, C11.1, C6.1, C7.1, C9.1, IC1.PIN, IC1.SPD, IC1.VBUS2, IC1.VDD2, IC2.!EXTMEM, IC2.VCC, IC2.VCC@1, R5.1
- net +5V: now also IC3.VH; no longer C5.1, IC3.VCC
- net AGND: now also C33.2, C34.2, CAN1.P$1, CN1.SHIELD, L7.2; no longer C1.2, C2.2, CN1.GND, D1.GND, IC1.GND1, IC1.GND1_2
- net DM4: no longer IC6.D-
- net DP4: no longer IC6.D+
- net GND: now also CN2.P$1, D2.A; no longer C4.2, C5.2
- net N$6: now also L3.1, R12.2; no longer C3.1, IC3.C1-
- net N$7: now also IC3.VL, L4.2; no longer C3.2, IC3.C1+
Other:
- note added: "CAN encloses everything"
- note added: "Inverted UART (Compliant with RS232)"
- note added: "LeaderTech SMS-462F"
- note removed: "Audio Codec"
- note removed: "RS232 Converter"
