File: Hardware/usb_hub_test.brd (EAGLE design)
At the start: 77.5 x 32.6 mm, 90 parts, among them CN1 54819-0519, CN2 TSW-120-08-L-S-RA, CN4 1-1734530-1, IC1 FT230XQ, IC2 TUSB2046BIRHBT, IC3 MAX3375, IC4 PIC24FJ128GA202-I/MM, IC5 FT230XQ, IC7 MAX3375

Commit message: Initial changes from v1 + started code
Parts:
- added C38: 10uF, rcl:C0805
- added C39: 1uF, rcl:C0402
- added R4: 15k, rcl:R0402
- moved CN5 3.14 mm to (6.80, 23.6), turned to 270 degrees
- moved R34 1.83 mm to (52.3, 22.2), turned to 180 degrees
- moved C2 0.91 mm to (52.4, 27.9), turned to 90 degrees
- moved CAN2 0.30 mm to (75.2, 3.37)
- moved C3 0.10 mm to (44.8, 22.5)
- moved R10 0.10 mm to (39.6, 22.5)
- moved R35 0.10 mm to (47.3, 22.5)
- moved R9 0.10 mm to (42.2, 22.5)
Connections:
- new net N$9: C39.1, IC2.4, R4.2
- new net PGC: IC4.19
- new net PGD: IC4.18
- net +3V3: now also IC2.10, IC2.14, IC2.18, IC2.22, R4.1; no longer IC2.4
- net +5V: now also C38.1, CN5.1
- net GND: now also C38.2, C39.2, U$1.5, U$1.TAB, U$1.TAB1
- net P3_RXD: now also U$1.1
- net P3_TXD: now also U$1.3
- net UART_FROM_CAT: now also IC4.14; no longer IC4.18
- net UART_FROM_WK: now also IC4.22; no longer IC4.21
- net UART_TO_CAT: now also IC4.15; no longer IC4.19
- net UART_TO_WK: now also IC4.23; no longer IC4.22
- net VBUS: no longer CN5.1
Routing:
- net DM1: track 53.8 -> 86.3 mm
- net DP1: track 52.7 -> 84.8 mm
- net +5V: track 63.0 -> 86.7 mm
- net N$189: track 7.34 -> 15.3 mm
- net P3_RXD: track 1.97 -> 7.68 mm
- net P3_TXD: track 1.97 -> 7.58 mm
- net PGD: track 0.00 -> 3.91 mm
- net +3V3: track 146.8 -> 150.5 mm
- net N$188: track 0.00 -> 2.67 mm
- net PGC: track 0.00 -> 2.01 mm
- net UART_TO_WK: track 21.2 -> 22.8 mm
- net UART_FROM_WK: track 22.3 -> 23.4 mm
- net !MCLR: track 14.9 -> 15.9 mm
- net UART_FROM_CAT: track 28.5 -> 29.4 mm
- net GND: track 39.7 -> 38.9 mm, vias 95 -> 116
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Other:
- outline, holes or cut-outs redrawn
- board text added: "!MCLR"
- board text added: "+5V"
- board text added: "232_DTR"
- board text added: "232_GND"
- board text added: "232_RTS"
- board text added: "232_RXD"
- board text added: "232_TXD"
- board text added: "ACC_ALC"
- board text added: "ACC_AUX"
- board text added: "ACC_BD0"
- board text added: "ACC_BD1"
- board text added: "ACC_BD2"
- board text added: "ACC_BD3"
- board text added: "ACC_DI0"
- board text added: "ACC_DI1"
- board text added: "ACC_DO0"
- board text added: "ACC_DO1"
- board text added: "ACC_GND"
- board text added: "ACC_KEY"
- board text added: "ACC_PTT"
- board text added: "ACC_PWR"
- board text added: "GND"
- board text added: "KIO3WUT MØWUT v0.12"
- board text added: "RX"
- board text added: "TX"

Commit message: Started work but fighting Microchip's stupid library
Parts:
- added R30, R31, R32, R33, R7, R8: 15k, rcl:R0402
Connections:
- new net N$11: IC2.15, R8.2
- new net N$14: IC2.16, R7.2
- net DM3: now also R30.2
- net DM4: now also R32.2
- net DP3: now also R31.2
- net DP4: now also R33.2
- net GND: now also R30.1, R31.1, R32.1, R33.1, R7.1, R8.1
