File: Hardware/usb_hub_test.brd (EAGLE design)
At the start: 77.5 x 32.6 mm, 102 parts, among them CN1 54819-0519, CN2 TSW-120-08-L-S-RA, CN3 48204-0001, CN4 1-1734530-1, IC1 FT230XQ, IC2 TUSB2046BIRHBT, IC3 IC_MAX3313, IC4 PIC24FJ128GA202-I/MM, IC5 FT230XQ

Commit message: renumbered parts, minor BOM update
Parts:
- removed R34: 2k2, rcl:R0402
- removed R35: 10k, rcl:R0402
- added R5, R6: 27, rcl:R0402
- C1, C35: value 100nF -> 1uF
- C10, C11, C29, C30, C32, C37: value 100nF -> 1nF
- C13, C15, C17, C19, C6, C7: value 1nF -> 100nF
- C14, C18: value 1nF -> 1uF
- C16, C4, C5: value 1nF -> 10uF; device rcl:C0402 -> rcl:C0805
- C2, C34: value 10uF -> 100nF; device rcl:C0805 -> rcl:C0402
- C25, C26, C31, C9: value 1uF -> 1nF
- C38: value 10uF -> 1nF; device rcl:C0805 -> rcl:C0402
- C39: value 1uF -> 10uF; device rcl:C0402 -> rcl:C0805
- C8: value 10uF -> 1uF; device rcl:C0805 -> rcl:C0402
- CN2: value TSW-120-08-L-S-RA -> 48204-0001; device m0wut:CONN_0.1_1X20 -> m0wut:CONN_USB_MOLEX_RA
- CN3: value 48204-0001 -> (none); device m0wut:CONN_USB_MOLEX_RA -> m0wut:USB_MICROB_WURTH
- CN4: value 1-1734530-1 -> TSW-120-08-L-S-RA; device m0wut:CONN_TE_DE-HD15 -> m0wut:CONN_0.1_1X20
- CN5: value (none) -> 1-1734530-1; device m0wut:USB_MICROB_WURTH -> m0wut:CONN_TE_DE-HD15
- IC1: value FT230XQ -> TUSB2046BIRHBT; device ftdichip:QFN16 -> texas:RHB_S-PQFP-N32
- IC2: value TUSB2046BIRHBT -> FT230XQ; device texas:RHB_S-PQFP-N32 -> ftdichip:QFN16
- IC3: value IC_MAX3313 -> FT230XQ; device m0wut:IC_UMAX10 -> ftdichip:QFN16
- IC5: value FT230XQ -> (none); device ftdichip:QFN16 -> m0wut:SOT23
- IC6: value (none) -> IC_MAX3313; device m0wut:SOT23 -> m0wut:IC_UMAX10
- L1: value (none) -> 100uH
- L4: value 100uH -> (none)
- R1, R2: value 1k5 -> 27
- R10: value 100k -> 27
- R12: value (none) -> 27
- R14: value 27 -> 1k5
- R15: value (none) -> 10k
- R16: value (none) -> 69k8
- R17: value 220 -> 100k
- R18: value 220 -> 2k2
- R23: value 220 -> 0R
- R29: value 137k -> 220
- R3: value 0R -> 27
- R30, R31: value (none) -> 220
- R32: value (none) -> 137k
- R4: value 15k -> 27
- R7: value (none) -> 15k
- R8: value (none) -> 1k5
- R9: value 69k8 -> 27
- RN1: value 2k2 -> 27
- RN3: value 27 -> 2k2
- moved C40 62.6 mm to (9.60, 25.9), turned to 270 degrees
- moved C41 56.1 mm to (9.60, 23.8), turned to 270 degrees
- moved C5 54.2 mm to (2.60, 19.2)
- moved L1 53.5 mm to (63.4, 22.4), turned to 0 degrees
- moved C35 53.1 mm to (62.5, 19.2), turned to 0 degrees
- moved L4 53.1 mm to (10.8, 29.6), turned to 270 degrees
- moved IC3 51.0 mm to (62.9, 26.4), turned to 0 degrees
- moved CN5 48.7 mm to (41.2, 0.00), flipped to the top, turned to 0 degrees
- moved C4 47.3 mm to (8.70, 29.6), turned to 270 degrees
- moved IC6 47.3 mm to (11.9, 24.3), turned to 270 degrees
- moved C1 41.7 mm to (73.4, 22.9), turned to 270 degrees
- moved C29 41.7 mm to (34.5, 13.3), turned to 0 degrees
- moved R30 39.5 mm to (30.7, 17.8), turned to 270 degrees
- moved R31 36.0 mm to (33.2, 17.8), turned to 270 degrees
- moved CN4 33.0 mm to (15.5, 20.6)
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- renumbered R33 to R12, U$1 to CN6
Connections:
- net !MCLR: now also C17.1, R15.1; no longer C3.1, R35.1
- net +3V3: now also C13.1, C14.1, C15.1, C2.1, C3.1, C34.1, C39.1, C6.1, C7.1, IC1.14, IC1.18, IC1.22, IC1.25, IC1.26, IC1.3, IC2.1, IC2.8, IC2.9, IC3.1, IC3.10, IC3.8, IC3.9, IC5.BOTTOM_RIGHT, R14.2, R15.2, R7.1, R8.2; no longer C10.1, C11.1, C25.1, C29.1, C30.1, C40.1, C41.1, C8.1, C9.1, IC1.1, IC1.8, IC1.9, IC2.14, IC2.18, IC2.22, IC2.25, IC2.26, IC2.3, IC5.1, IC5.10, IC5.8, IC5.9, IC6.BOTTOM_RIGHT, R1.2, R2.2, R35.2, R4.1
- net +5V: now also C18.1, C19.1, C4.1, C5.1, CN2.1, IC5.TOP, L1.2, L4.1, R16.2, R18.2, RN3.1, RN3.2, RN3.3; no longer C31.1, C32.1, C34.1, C38.1, CN5.1, IC6.TOP, L4.2, L6.1, R34.2, R9.2, RN1.1, RN1.2, RN1.3
- net 232_DTR: now also CN4.P$2; no longer CN2.P$2
- net 232_FROM_P3: now also L6.2; no longer L5.2
- net 232_RTS: now also CN4.P$4; no longer CN2.P$4
- net 232_RXD: now also C38.1, CN4.P$5, L3.2; no longer C28.1, CN2.P$5, L2.2
- net 232_TO_P3: now also L5.2; no longer L1.2
- net 232_TXD: now also C37.1, CN4.P$3, L2.2; no longer C27.1, CN2.P$3, L3.2
- net 5V_IN: now also C35.1, CN4.P$20, L1.1; no longer C26.1, CN2.P$20, L4.1
- net ACC_ALC: now also CN4.P$12, R16.1, R17.2, R32.1; no longer CN2.P$12, R10.2, R29.1, R9.1
- net ACC_AUX: now also CN4.P$15, R20.1; no longer CN2.P$15, R18.1
- net ACC_BND0: now also CN4.P$7, R30.1, RN3.1A; no longer CN2.P$7, R27.1, RN1.1A
- net ACC_BND1: now also CN4.P$14, R18.1, R21.1; no longer CN2.P$14, R19.1, R34.1
- net ACC_BND2: now also CN4.P$9, R27.1, RN3.3A; no longer CN2.P$9, R24.1, RN1.3A
- net ACC_BND3: now also CN4.P$8, R31.1, RN3.2A; no longer CN2.P$8, R28.1, RN1.2A
- net ACC_COMMON: now also C20.1, CN5.12, CN5.5, R23.2; no longer C33.1, CN4.12, CN4.5, R3.2
- net ACC_DI0: now also CN4.P$16, R19.1; no longer CN2.P$16, R17.1
- net ACC_DI1: now also CN4.P$17, R25.1; no longer CN2.P$17, R22.1
- net ACC_DO0: now also CN4.P$18, R24.1; no longer CN2.P$18, R21.1
- net ACC_DO1: now also CN4.P$19, R29.1; no longer CN2.P$19, R26.1
- net ACC_KEY: now also CN4.P$10, R28.1; no longer CN2.P$10, R25.1
- net ACC_PTT: now also CN4.P$13, R22.1; no longer CN2.P$13, R20.1
- net ACC_PWR: now also CN4.P$11, R26.1; no longer CN2.P$11, R23.1
- net AGND: now also C25.2, C26.2, C29.2, C30.2, C31.2, C32.2, C37.2, C38.2, CN5.16, CN5.17; no longer C12.2, C13.2, C14.2, C15.2, C16.2, C17.2, C18.2, C19.2, CN4.16, CN4.17
- net ALC_X: now also C33.1, CN5.15, R32.2; no longer C24.1, CN4.15, R29.2
- net ASDF: now also L2.1; no longer L3.1
- net AUX_X: now also C22.1, CN5.2, R20.2; no longer C13.1, CN4.2, R18.2
- net BND0_X: now also C31.1, CN5.13, R30.2; no longer C22.1, CN4.13, R27.2
- net BND1_X: now also C23.1, CN5.3, R21.2; no longer C14.1, CN4.3, R19.2
- net BND2_X: now also C28.1, CN5.9, R27.2; no longer C19.1, CN4.9, R24.2
- net BND3_X: now also C32.1, CN5.14, R31.2; no longer C23.1, CN4.14, R28.2
- net D+_P: now also R1.1; no longer R11.1
- net DIG0_X: now also C21.1, CN5.1, R19.2; no longer C12.1, CN4.1, R17.2
- net DIG1_X: now also C26.1, CN5.7, R25.2; no longer C17.1, CN4.7, R22.2
- net DIGO1_X: now also C30.1, CN5.11, R29.2; no longer C21.1, CN4.11, R26.2
- net DIGO_X: now also C25.1, CN5.6, R24.2; no longer C16.1, CN4.6, R21.2
- net DM0: now also IC1.2, R2.2; no longer IC2.2, R14.2
- net DM1: now also CN2.2, R3.1, RN1.1A; no longer CN3.2, R7.1, RN2.1A
- net DM2: now also CN3.2, R5.1, RN1.3A; no longer CN5.2, R15.1, RN2.3A
- net DM3: now also IC3.7, RN2.1A; no longer IC5.7, RN3.1A
- net DM4: now also IC2.7, R10.2, RN2.3A; no longer IC1.7, R31.2, RN3.3A
- net DP0: now also IC1.1, R1.2, R8.1; no longer IC2.1, R11.2, R13.1
- net DP1: now also CN2.3, R4.1, RN1.2A; no longer CN3.3, R8.1, RN2.2A
- net DP2: now also CN3.3, R6.1, RN1.4A; no longer CN5.3, R16.1, RN2.4A
- net DP3: now also IC3.6, R11.2, R14.1, RN2.2A; no longer IC5.6, R2.1, R32.2, RN3.2A
- net DP4: now also IC2.6, R13.1, R9.2, RN2.4A; no longer IC1.6, R1.1, R30.2, RN3.4A
- net GND: now also C12.2, C13.2, C14.2, C15.2, C16.2, C17.2, C18.2, C19.2, C35.2, CN2.4, CN2.P$2, CN2.P$3, CN2.P$4, CN2.P$5, CN3.5, CN3.GND1, CN3.GND2, CN3.GND3, CN3.GND4, CN4.P$1, CN4.P$6, IC1.27, IC1.28, IC1.31, IC1.6, IC1.7, IC1.8, IC1.EXP, IC2.13, IC2.3, IC2.P$1, IC2.P$2, IC2.P$3, IC2.P$4, IC2.TAB, IC3.13, IC3.3, IC3.P$1, IC3.P$2, IC3.P$3, IC3.P$4, IC3.TAB, IC5.BOTTOM_LEFT, IC6.10, R17.1, R23.1, RN1.1, RN1.2, RN1.3, RN1.4; no longer C25.2, C26.2, C29.2, C30.2, C31.2, C32.2, C37.2, C38.2, C41.2, CN2.P$1, CN2.P$6, CN3.P$2, CN3.P$3, CN3.P$4, CN3.P$5, CN5.4, CN5.5, CN5.GND1, CN5.GND2, CN5.GND3, CN5.GND4, IC1.13, IC1.3, IC1.P$1, IC1.P$2, IC1.P$3, IC1.P$4, IC1.TAB, IC2.27, IC2.28, IC2.31, IC2.6, IC2.7, IC2.8, IC2.EXP, IC3.10, IC5.13, IC5.3, IC5.P$1, IC5.P$2, IC5.P$3, IC5.P$4, IC5.TAB, IC6.BOTTOM_LEFT, R10.1, R3.1, RN3.1, RN3.2, RN3.3, RN3.4
- net KEY_X: now also C29.1, CN5.10, R28.2; no longer C20.1, CN4.10, R25.2
- net N$1: now also IC1.23, R10.1; no longer IC2.23, R31.1
- net N$10: now also IC1.29; no longer IC2.29
- net N$11: now also IC1.15, R5.2; no longer IC2.15, R15.2
- net N$12: now also IC1.11, R3.2; no longer IC2.11, R7.2
- net N$13: now also IC1.12, R4.2; no longer IC2.12, R8.2
- net N$14: now also IC1.16, R6.2; no longer IC2.16, R16.2
- net N$15: now also C42.1, IC6.8; no longer C37.1, IC3.8
- net N$16: now also IC1.20, R11.1; no longer IC2.20, R32.1
- net N$17: now also IC1.19; no longer IC2.19
- net N$2: now also C16.1; no longer C2.1
- net N$20: now also R2.1; no longer R14.1
- net N$3: now also IC1.24, R9.1; no longer IC2.24, R30.1
- net N$4: now also C40.1, IC6.1, L4.2; no longer C42.1, IC3.1, L6.2
- net N$6: now also C41.1, IC6.2; no longer C35.1, IC3.2
- net N$7: now also C41.2, IC6.9; no longer C35.2, IC3.9
- net N$8: now also IC1.30; no longer IC2.30
- net N$9: now also C8.1, IC1.4, R7.2; no longer C39.1, IC2.4, R4.2
- net PTT_X: now also C24.1, CN5.4, R22.2; no longer C15.1, CN4.4, R20.2
- net PWR_X: now also C27.1, CN5.8, R26.2; no longer C18.1, CN4.8, R23.2
- net SADF: now also L3.1; no longer L2.1
- net UART_FROM_CAT: now also C9.1, IC2.2; no longer C5.1, IC1.2
- net UART_FROM_P3: now also IC6.5; no longer IC3.5
- net UART_FROM_WK: now also C11.1, IC3.2; no longer C7.1, IC5.2
- net UART_TO_CAT: now also C12.1, IC2.15; no longer C4.1, IC1.15
- net UART_TO_P3: now also IC6.4; no longer IC3.4
- net UART_TO_WK: now also C10.1, IC3.15; no longer C6.1, IC5.15
- net WTRE: now also IC6.7, L5.1; no longer IC3.7, L1.1
- net Y5W4: now also IC6.6, L6.1; no longer IC3.6, L5.1

Commit message: minor code fixes
Parts:
- L4: value (none) -> 100uH
- RN1, RN2: value 27 -> 15k
Changed lines of the file:
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@@
 <attribute name="VALUE" x="69.1" y="12.1" size="1.016" layer="28" font="vector" rot="MR270" align="center"/>
 </element>
-<element name="RN2" library="m0wut" package="R_BOURNS_CAY16-J4" value="27" x="68.05" y="23.15" smashed="yes" rot="MR180"/>
+<element name="RN2" library="m0wut" package="R_BOURNS_CAY16-J4" value="15k" x="68.05" y="23.15" smashed="yes" rot="MR180"/>
 <element name="C6" library="rcl" package="C0402" value="100nF" x="71.85" y="19.5" smashed="yes" rot="MR180">
 <attribute name="VALUE" x="71.85" y="20.9" size="1.016" layer="28" font="vector" rot="MR180" align="center"/>
@@
 <attribute name="VALUE" x="65.345" y="20.55" size="1.016" layer="28" font="vector" rot="MR90" align="center"/>
 </element>
-<element name="RN1" library="m0wut" package="R_BOURNS_CAY16-J4" value="27" x="58.9" y="9.6" smashed="yes" rot="MR0"/>
+<element name="RN1" library="m0wut" package="R_BOURNS_CAY16-J4" value="15k" x="58.9" y="9.6" smashed="yes" rot="MR0"/>
 <element name="Q1" library="adafruit" package="SOT23" value="" x="28.2" y="27.3" smashed="yes" rot="MR270">
 <attribute name="VALUE" x="31.375" y="27.3" size="1.27" layer="28" font="vector" rot="MR270" align="center"/>
@@
 <attribute name="VALUE" x="14.432" y="17.8" size="1.27" layer="28" font="vector" rot="MR270" align="center"/>
 </element>
-<element name="L4" library="m0wut" package="R0805" value="" x="10.8" y="29.6" smashed="yes" rot="MR270">
+<element name="L4" library="m0wut" package="R0805" value="100uH" x="10.8" y="29.6" smashed="yes" rot="MR270">
 <attribute name="VALUE" x="12.832" y="29.6" size="1.27" layer="28" font="vector" rot="MR270" align="center"/>
 </element>
