File: Hardware/usb_hub_test.sch (EAGLE design)
At the start: 78 parts, among them CN1 54819-0519, CN2 TSW-120-08-L-S-RA, CN3 1734354-1, CN4 1-1734530-1, IC1 ADUM3160BRWZ, IC2 TUSB2046BIRHBT, IC4 FT2232D

Commit message: nearly there...
Parts:
- removed CAN1: SHIELDING_CAN, m0wut:SHIELDING_CAN
- removed CN3: 1734354-1, m0wut:CONN_TE_DB9
- removed L7: 100uH, m0wut:INDUCTOR
- removed R4, R7: 24, rcl:R-EU_R0402
- removed R8: 69k8, rcl:R-EU_R0402
- added C3, C35, C37: 100nF, rcl:C-EUC0402
- added C36: 1uF, rcl:C-EUC0402
- added C4, C5: 1nF, rcl:C-EUC0402
- added CAN2: CAN_MASTECH, m0wut:CAN_MASTECH
- added CN5: (no value), m0wut:USBOTG_VERTICAL
- added D3: BZT52C4V7-7-F, adafruit:DIODESOD-123
- added IC5: FT230XQ, ftdichip:FT230XQ
- added IC6: (no value), m0wut:MCP1700
- added IC7: MAX3375, m0wut:IC_MAX3375
- added R13: 1k5, rcl:R-EU_R0402
- added R34: 2k2, rcl:R-EU_R0402
- added R35: 10k, rcl:R-EU_R0402
- added RN2: (no value), m0wut:R_BOURNS_CAY16-J4
- added U$1: SS-640810S-A-NF-A111, m0wut:CONN_RJ45_SHIELDEDSTEWART_SHORTER
- added X1: (no value), m0wut:XTAL_MURATA_3-PIN-RES
- C1: value 1uF -> 100nF
- C2, C8: value 1uF -> 10uF; device rcl:C-EUC0402 -> rcl:C-EUC0805
- C26: value 33nF -> 1uF
- C27, C28, C7: value 100nF -> 1nF
- C6: value 1uF -> 1nF
- CN1: device m0wut:USBMOLEX_MINI -> m0wut:USBMUSB
- D2: value BZT52C3V0-7-F -> BZT52C4V7-7-F
- IC1: value ADUM3160BRWZ -> FT230XQ; device m0wut:ADUM3160BRWZ -> ftdichip:FT230XQ
- IC3: value (none) -> MAX3375
- IC4: value FT2232D -> PIC24FJ128GA202-I/MM; device ftdichip-3:FT2232D -> m0wut:PIC24FJ128GA202-I/MM
- R1, R2: value 24 -> 1k5
- R10: value 24 -> 100k
- R11: value 24 -> 27
- R14: value 1k5 -> 27
- R15: value 470 -> 27
- R16: value 10k -> 27
- R17, R18, R19, R20, R21, R22, R23, R24, R25, R26, R27, R28, R29: device rcl:R-EU_R0805 -> rcl:R-EU_R0402
- R3: value 24 -> 220
- R6: value 24 -> 15k
- R9: value 100k -> 69k8
Connections:
- removed net 3V3_HUB: C10.1, C11.1, C9.1, IC2.!EXTMEM, IC2.VCC, IC2.VCC@1, L6.2, R5.1
- removed net 6MHZ_FT: IC4.XTIN
- removed net 6MHZ_HUB: IC2.XTAL1
- removed net ACC_COM: CN2.P$6, L1.1
- removed net AGND: C12.2, C13.2, C14.2, C15.2, C16.2, C17.2, C18.2, C19.2, C20.2, C21.2, C22.2, C23.2, C24.2, C33.2, C34.2, CAN1.P$1, CN1.SHIELD, CN3.TAB, CN4.TAB, L7.2
- removed net CAT_232_TO_PIC: IC4.ADBUS0
- removed net CAT_PIC_TO_232: IC4.ADBUS1
- removed net D+: D1.LEFT, IC1.UD+, R1.2
- removed net D-: D1.RIGHT, IC1.UD-, R2.2
- removed net DM2: IC4.D-, R10.1
- removed net DP2: IC4.D+, R11.1, R14.2
- removed net N$11: IC1.DD+, R4.1
- removed net N$14: IC2.DM2, R10.2
- removed net N$15: IC2.DP2, R11.2
- removed net N$18: C33.1, CN3.2, L2.2
- removed net N$19: C6.1, C7.1, IC1.PIN, IC1.SPD, IC1.VBUS2, IC1.VDD2, L5.1
- removed net N$33: C27.1, IC4.AVCC, R15.1
- removed net N$37: IC4.EEDATA, R16.2
- removed net N$9: C2.1, IC1.PDEN, IC1.SPU, IC1.VDD1
- removed net USB4_N: IC2.DM4, R7.1
- removed net USB4_P: IC2.DP4, R6.1
- removed net USB_IN_GND: C1.2, C2.2, CN1.GND, D1.GND, IC1.GND1, IC1.GND1_2, L7.1
- removed net VCC: C1.1, CN1.VBUS, D1.V+, IC1.VBUS1
- removed net VDD: C26.1, IC4.3V3OUT, R14.1
- removed net WK_232_TO_PIC: IC4.BDBUS0
- removed net WK_PIC_TO_232: IC4.BDBUS1
- new net !MCLR: C3.1, IC4.!MCLR, R35.1
- new net D+_P: CN1.D+, R11.1
- new net DM1: CN5.D-, R15.1, R5.2
- new net DM3: IC5.USBDM, RN2.4A
- new net DP1: CN5.D+, R16.1, R6.2
- new net DP3: IC5.USBDP, R2.1, RN2.3A
- new net N$20: CN1.D-, R14.1
- new net N$5: IC7.OH, L5.1
- new net N$8: IC2.XTAL1, X1.XTAL1
- new net P3_RXD: C27.1, L5.2
- new net P3_TXD: C28.1, L6.2
- new net UART_FROM_CAT: C5.1, IC1.RXD, IC4.RB10
- new net UART_FROM_K3: IC3.OL, IC4.RB0
- new net UART_FROM_P3: IC4.RB2, IC7.OL
- new net UART_FROM_WK: C7.1, IC4.RB13, IC5.RXD
- new net UART_TO_CAT: C4.1, IC1.TXD, IC4.RB11
- new net UART_TO_K3: IC3.IL, IC4.RB1
- new net UART_TO_P3: IC4.RB3, IC7.IL
- new net UART_TO_WK: C6.1, IC4.RB14, IC5.TXD
- new net VBUS: CN1.VBUS, CN5.VBUS, D1.V+
- net +3V3: now also C1.1, C10.1, C11.1, C25.1, C29.1, C30.1, C35.1, C8.1, C9.1, IC1.!RESET, IC1.3V3OUT, IC1.VCC, IC1.VCCIO, IC2.!EXTMEM, IC2.!RESET, IC2.VCC, IC2.VCC@1, IC3.EN, IC3.VL, IC4.VDD, IC5.!RESET, IC5.3V3OUT, IC5.VCC, IC5.VCCIO, IC6.VO, IC7.EN, IC7.VL, R1.2, R13.2, R2.2, R35.2; no longer L4.1, L5.2, L6.1
- net +5V: now also C36.1, C37.1, IC6.VI, IC7.VH, L4.2, R34.2, R9.2; no longer C25.1, C28.1, C29.1, C30.1, IC4.-RESET, IC4.SI/WUA, IC4.SI/WUB, IC4.VCC@1, IC4.VCC@2, IC4.VCCIOA, IC4.VCCIOB, R15.2, R16.1, R8.2, RN1.4
- net 232_RXD: now also C33.1, L2.2
- net 232_TXD: now also C34.1, L3.2
- net 5V_IN: now also C26.1, L4.1
- net ACC_ALC: now also R10.2, R9.1; no longer R8.1, R9.2
- net ACC_BND1: now also R34.1; no longer RN1.4A
- net DM0: now also D1.LEFT, R14.2; no longer R3.2
- net DM4: now also IC1.USBDM, RN2.2A; no longer R7.2
- net DP0: now also D1.RIGHT, R11.2, R13.1; no longer R4.2
- net DP4: now also IC1.USBDP, R1.1, RN2.1A; no longer R6.2
- net GND: now also C1.2, C12.2, C13.2, C14.2, C15.2, C16.2, C17.2, C18.2, C19.2, C2.2, C20.2, C21.2, C22.2, C23.2, C24.2, C3.2, C33.2, C34.2, C35.2, C36.2, C37.2, C4.2, C5.2, CAN2.P$1, CN1.GND, CN1.SHIELD, CN2.P$6, CN4.TAB, CN5.GND, CN5.ID, CN5.SHIELD, D1.GND, D3.A, IC1.GND, IC1.GND@1, IC4.VSS, IC5.GND, IC5.GND@1, IC6.GND, IC7.GND, L1.1, R10.1, R5.1, R6.1, X1.CAN; no longer CN3.5, IC1.GND2, IC1.GND2_2, IC4.AGND, IC4.GND@1, IC4.GND@2, IC4.GND@3, IC4.GND@4, IC4.TEST, R9.1
- net N$1: now also IC2.DM4, RN2.2; no longer CN1.D+, R1.1
- net N$10: now also IC2.XTAL2, X1.XTAL2; no longer IC1.DD-, R3.1
- net N$12: now also R15.2
- net N$13: now also R16.2
- net N$16: now also RN2.3
- net N$17: now also RN2.4
- net N$2: now also C2.1, IC4.VCAP; no longer CN1.D-, R2.1
- net N$3: now also IC2.DP4, RN2.1; no longer C8.1, IC2.!RESET, R5.2
- net N$4: now also D3.C, IC7.IH, R3.1; no longer C34.1, CN3.3, L3.2
- net N$7: now also L6.1, R3.2; no longer IC3.VL, L4.2
Other:
- note added: "Pickit 3"
- note added: "Power Supply"
- note added: "TO FT220_2"
- note added: "TO FT230_1"
- note removed: "CAN encloses everything"
- note removed: "LeaderTech SMS-462F"
- note removed: "TO CODEC"
- note removed: "TO FT2232"
- note removed: "USB0 (Not Used)"
- note removed: "USB3 (Not Used)"

Commit message: Initial changes from v1 + started code
Parts:
- added C38: 10uF, rcl:C-EUC0805
- added C39: 1uF, rcl:C-EUC0402
- added R4: 15k, rcl:R-EU_R0402
Connections:
- new net N$9: C39.1, IC2.!RESET, R4.2
- new net PGC: IC4.RB11
- new net PGD: IC4.RB10
- net +3V3: now also IC2.!OVRCUR1, IC2.!OVRCUR2, IC2.!OVRCUR3, IC2.!OVRCUR4, R4.1; no longer IC2.!RESET
- net +5V: now also C38.1, CN5.VBUS
- net GND: now also C38.2, C39.2, U$1.5, U$1.TAB
- net P3_RXD: now also U$1.1
- net P3_TXD: now also U$1.3
- net UART_FROM_CAT: now also IC4.RB8; no longer IC4.RB10
- net UART_FROM_WK: now also IC4.RB14; no longer IC4.RB13
- net UART_TO_CAT: now also IC4.RB9; no longer IC4.RB11
- net UART_TO_WK: now also IC4.RB15; no longer IC4.RB14
- net VBUS: no longer CN5.VBUS

Commit message: Started work but fighting Microchip's stupid library
Parts:
- added R30, R31, R32, R33, R7, R8: 15k, rcl:R-EU_R0402
Connections:
- new net N$11: IC2.DM2, R8.2
- new net N$14: IC2.DP2, R7.2
- net DM3: now also R30.2
- net DM4: now also R32.2
- net DP3: now also R31.2
- net DP4: now also R33.2
- net GND: now also R30.1, R31.1, R32.1, R33.1, R7.1, R8.1
Other:
- note removed: "TO FT220_2"
- note removed: "TO FT230_1"
- moved on the sheet: RN2
Changed lines of the file:
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@@
 <part name="C39" library="rcl" deviceset="C-EU" device="C0402" value="1uF"/>
 <part name="GND39" library="supply1" deviceset="GND" device=""/>
+<part name="R7" library="rcl" deviceset="R-EU_" device="R0402" value="15k"/>
+<part name="R8" library="rcl" deviceset="R-EU_" device="R0402" value="15k"/>
+<part name="GND40" library="supply1" deviceset="GND" device=""/>
+<part name="GND41" library="supply1" deviceset="GND" device=""/>
+<part name="R30" library="rcl" deviceset="R-EU_" device="R0402" value="15k"/>
+<part name="R31" library="rcl" deviceset="R-EU_" device="R0402" value="15k"/>
+<part name="R32" library="rcl" deviceset="R-EU_" device="R0402" value="15k"/>
+<part name="R33" library="rcl" deviceset="R-EU_" device="R0402" value="15k"/>
+<part name="GND42" library="supply1" deviceset="GND" device=""/>
+<part name="GND43" library="supply1" deviceset="GND" device=""/>
+<part name="GND44" library="supply1" deviceset="GND" device=""/>
+<part name="GND45" library="supply1" deviceset="GND" device=""/>
 </parts>
 <sheets>
@@
 <text x="218.44" y="15.24" size="2.54" layer="94">Dan M0WUT</text>
 <text x="218.44" y="10.16" size="2.54" layer="94">USB Hub</text>
-<text x="226.06" y="111.76" size="1.778" layer="95">TO FT220_2</text>
-<text x="226.06" y="86.36" size="1.778" layer="95">TO FT230_1</text>
 </plain>
 <instances>
@@
 <instance part="CN5" gate="G$1" x="53.34" y="93.98"/>
 <instance part="GND23" gate="1" x="53.34" y="76.2"/>
-<instance part="RN2" gate="G$1" x="215.9" y="96.52"/>
+<instance part="RN2" gate="G$1" x="203.2" y="96.52"/>
 <instance part="P+4" gate="1" x="68.58" y="119.38"/>
 <instance part="C38" gate="G$1" x="78.74" y="111.76"/>
 <instance part="GND38" gate="1" x="78.74" y="101.6"/>
 <instance part="+3V10" gate="G$1" x="109.22" y="111.76"/>
-<instance part="+3V11" gate="G$1" x="109.22" y="88.9"/>
+<instance part="+3V11" gate="G$1" x="96.52" y="88.9"/>
 <instance part="+3V12" gate="G$1" x="180.34" y="91.44"/>
 <instance part="+3V13" gate="G$1" x="187.96" y="109.22"/>
@@
 <instance part="C39" gate="G$1" x="91.44" y="119.38"/>
 <instance part="GND39" gate="1" x="91.44" y="109.22"/>
+<instance part="R7" gate="G$1" x="127" y="78.74" rot="R90"/>
+<instance part="R8" gate="G$1" x="119.38" y="78.74" rot="R90"/>
+<instance part="GND40" gate="1" x="119.38" y="68.58"/>
+<instance part="GND41" gate="1" x="127" y="68.58"/>
+<instance part="R30" gate="G$1" x="210.82" y="81.28" rot="R90"/>
+<instance part="R31" gate="G$1" x="218.44" y="81.28" rot="R90"/>
+<instance part="R32" gate="G$1" x="226.06" y="81.28" rot="R90"/>
+<instance part="R33" gate="G$1" x="233.68" y="81.28" rot="R90"/>
+<instance part="GND42" gate="1" x="210.82" y="71.12"/>
+<instance part="GND43" gate="1" x="218.44" y="71.12"/>
+<instance part="GND44" gate="1" x="226.06" y="71.12"/>
+<instance part="GND45" gate="1" x="233.68" y="71.12"/>
 </instances>
 <busses>
@@
 <wire x1="91.44" y1="114.3" x2="91.44" y2="111.76" width="0.1524" layer="91"/>
 </segment>
+<segment>
+<pinref part="R8" gate="G$1" pin="1"/>
+<pinref part="GND40" gate="1" pin="GND"/>
+<wire x1="119.38" y1="73.66" x2="119.38" y2="71.12" width="0.1524" layer="91"/>
+</segment>
+<segment>
+<pinref part="R7" gate="G$1" pin="1"/>
+<pinref part="GND41" gate="1" pin="GND"/>
+<wire x1="127" y1="73.66" x2="127" y2="71.12" width="0.1524" layer="91"/>
+</segment>
+<segment>
+<pinref part="GND42" gate="1" pin="GND"/>
+<pinref part="R30" gate="G$1" pin="1"/>
+<wire x1="210.82" y1="73.66" x2="210.82" y2="76.2" width="0.1524" layer="91"/>
+</segment>
+<segment>
+<pinref part="GND43" gate="1" pin="GND"/>
+<pinref part="R31" gate="G$1" pin="1"/>
+<wire x1="218.44" y1="73.66" x2="218.44" y2="76.2" width="0.1524" layer="91"/>
+</segment>
+<segment>
+<pinref part="GND44" gate="1" pin="GND"/>
+<pinref part="R32" gate="G$1" pin="1"/>
+<wire x1="226.06" y1="73.66" x2="226.06" y2="76.2" width="0.1524" layer="91"/>
+</segment>
+<segment>
+<pinref part="GND45" gate="1" pin="GND"/>
+<pinref part="R33" gate="G$1" pin="1"/>
+<wire x1="233.68" y1="73.66" x2="233.68" y2="76.2" width="0.1524" layer="91"/>
+</segment>
 </net>
 <net name="N$12" class="0">
@@
 <wire x1="172.72" y1="101.6" x2="187.96" y2="101.6" width="0.1524" layer="91"/>
 <pinref part="RN2" gate="G$1" pin="3"/>
-<wire x1="208.28" y1="96.52" x2="187.96" y2="96.52" width="0.1524" layer="91"/>
+<wire x1="195.58" y1="96.52" x2="187.96" y2="96.52" width="0.1524" layer="91"/>
 <wire x1="187.96" y1="96.52" x2="187.96" y2="101.6" width="0.1524" layer="91"/>
 </segment>
@@
 <wire x1="172.72" y1="99.06" x2="185.42" y2="99.06" width="0.1524" layer="91"/>
 <pinref part="RN2" gate="G$1" pin="4"/>
-<wire x1="208.28" y1="93.98" x2="185.42" y2="93.98" width="0.1524" layer="91"/>
+<wire x1="195.58" y1="93.98" x2="185.42" y2="93.98" width="0.1524" layer="91"/>
 <wire x1="185.42" y1="93.98" x2="185.42" y2="99.06" width="0.1524" layer="91"/>
 </segment>
@@
 <segment>
 <pinref part="IC2" gate="G$1" pin="!OVRCUR2"/>
-<wire x1="121.92" y1="99.06" x2="116.84" y2="99.06" width="0.1524" layer="91"/>
-<wire x1="116.84" y1="99.06" x2="116.84" y2="83.82" width="0.1524" layer="91"/>
+<wire x1="121.92" y1="99.06" x2="114.3" y2="99.06" width="0.1524" layer="91"/>
+<wire x1="114.3" y1="99.06" x2="114.3" y2="86.36" width="0.1524" layer="91"/>
 <pinref part="+3V11" gate="G$1" pin="+3V3"/>
-<wire x1="116.84" y1="83.82" x2="109.22" y2="83.82" width="0.1524" layer="91"/>
-<wire x1="109.22" y1="83.82" x2="109.22" y2="86.36" width="0.1524" layer="91"/>
+<wire x1="114.3" y1="86.36" x2="96.52" y2="86.36" width="0.1524" layer="91"/>
 </segment>
 <segment>
@@
 <segment>
 <pinref part="RN2" gate="G$1" pin="2"/>
-<wire x1="208.28" y1="99.06" x2="193.04" y2="99.06" width="0.1524" layer="91"/>
+<wire x1="195.58" y1="99.06" x2="193.04" y2="99.06" width="0.1524" layer="91"/>
 <wire x1="193.04" y1="99.06" x2="193.04" y2="109.22" width="0.1524" layer="91"/>
 <pinref part="IC2" gate="G$1" pin="DM4"/>
@@
 <segment>
 <pinref part="RN2" gate="G$1" pin="1"/>
-<wire x1="208.28" y1="101.6" x2="195.58" y2="101.6" width="0.1524" layer="91"/>
 <wire x1="195.58" y1="101.6" x2="195.58" y2="111.76" width="0.1524" layer="91"/>
 <pinref part="IC2" gate="G$1" pin="DP4"/>
@@
 <segment>
 <pinref part="RN2" gate="G$1" pin="1A"/>
-<wire x1="223.52" y1="101.6" x2="236.22" y2="101.6" width="0.1524" layer="91"/>
-<label x="231.14" y="101.6" size="1.778" layer="95"/>
+<wire x1="210.82" y1="101.6" x2="233.68" y2="101.6" width="0.1524" layer="91"/>
+<label x="243.84" y="101.6" size="1.778" layer="95"/>
+<pinref part="R33" gate="G$1" pin="2"/>
+<wire x1="233.68" y1="101.6" x2="248.92" y2="101.6" width="0.1524" layer="91"/>
+<wire x1="233.68" y1="86.36" x2="233.68" y2="101.6" width="0.1524" layer="91"/>
+<junction x="233.68" y="101.6"/>
 </segment>
 </net>
@@
 <segment>
 <pinref part="RN2" gate="G$1" pin="2A"/>
-<wire x1="223.52" y1="99.06" x2="236.22" y2="99.06" width="0.1524" layer="91"/>
-<label x="231.14" y="99.06" size="1.778" layer="95"/>
+<wire x1="210.82" y1="99.06" x2="226.06" y2="99.06" width="0.1524" layer="91"/>
+<label x="243.84" y="99.06" size="1.778" layer="95"/>
+<pinref part="R32" gate="G$1" pin="2"/>
+<wire x1="226.06" y1="99.06" x2="248.92" y2="99.06" width="0.1524" layer="91"/>
+<wire x1="226.06" y1="86.36" x2="226.06" y2="99.06" width="0.1524" layer="91"/>
+<junction x="226.06" y="99.06"/>
 </segment>
 </net>
@@
 <segment>
 <pinref part="RN2" gate="G$1" pin="3A"/>
-<wire x1="223.52" y1="96.52" x2="236.22" y2="96.52" width="0.1524" layer="91"/>
-<label x="231.14" y="96.52" size="1.778" layer="95"/>
+<wire x1="210.82" y1="96.52" x2="218.44" y2="96.52" width="0.1524" layer="91"/>
+<label x="243.84" y="96.52" size="1.778" layer="95"/>
+<pinref part="R31" gate="G$1" pin="2"/>
+<wire x1="218.44" y1="96.52" x2="248.92" y2="96.52" width="0.1524" layer="91"/>
+<wire x1="218.44" y1="86.36" x2="218.44" y2="96.52" width="0.1524" layer="91"/>
+<junction x="218.44" y="96.52"/>
 </segment>
 </net>
@@
 <segment>
 <pinref part="RN2" gate="G$1" pin="4A"/>
-<wire x1="223.52" y1="93.98" x2="236.22" y2="93.98" width="0.1524" layer="91"/>
-<label x="231.14" y="93.98" size="1.778" layer="95"/>
+<wire x1="210.82" y1="93.98" x2="248.92" y2="93.98" width="0.1524" layer="91"/>
+<label x="243.84" y="93.98" size="1.778" layer="95"/>
+<pinref part="R30" gate="G$1" pin="2"/>
+<wire x1="210.82" y1="86.36" x2="210.82" y2="93.98" width="0.1524" layer="91"/>
+<junction x="210.82" y="93.98"/>
 </segment>
 </net>
@@
 </segment>
 </net>
+<net name="N$11" class="0">
+<segment>
+<pinref part="IC2" gate="G$1" pin="DM2"/>
+<pinref part="R8" gate="G$1" pin="2"/>
+<wire x1="121.92" y1="96.52" x2="119.38" y2="96.52" width="0.1524" layer="91"/>
+<wire x1="119.38" y1="96.52" x2="119.38" y2="83.82" width="0.1524" layer="91"/>
+</segment>
+</net>
+<net name="N$14" class="0">
+<segment>
+<pinref part="R7" gate="G$1" pin="2"/>
+<wire x1="127" y1="83.82" x2="127" y2="86.36" width="0.1524" layer="91"/>
+<pinref part="IC2" gate="G$1" pin="DP2"/>
+<wire x1="127" y1="86.36" x2="121.92" y2="86.36" width="0.1524" layer="91"/>
+<wire x1="121.92" y1="86.36" x2="121.92" y2="93.98" width="0.1524" layer="91"/>
+</segment>
+</net>
