File: Hardware/usb_hub_test.sch (EAGLE design)
At the start: 102 parts, among them CN1 54819-0519, CN2 TSW-120-08-L-S-RA, CN3 48204-0001, CN4 1-1734530-1, IC1 FT230XQ, IC2 TUSB2046BIRHBT, IC3 IC_MAX3313, IC4 PIC24FJ128GA202-I/MM, IC5 FT230XQ

Commit message: renumbered parts, minor BOM update
Parts:
- removed R34: 2k2, rcl:R-EU_R0402
- removed R35: 10k, rcl:R-EU_R0402
- added R5, R6: 27, rcl:R-EU_R0402
- C1, C35: value 100nF -> 1uF
- C10, C11, C29, C30, C32, C37: value 100nF -> 1nF
- C13, C15, C17, C19, C6, C7: value 1nF -> 100nF
- C14, C18: value 1nF -> 1uF
- C16, C4, C5: value 1nF -> 10uF; device rcl:C-EUC0402 -> rcl:C-EUC0805
- C2, C34: value 10uF -> 100nF; device rcl:C-EUC0805 -> rcl:C-EUC0402
- C25, C26, C31, C9: value 1uF -> 1nF
- C38: value 10uF -> 1nF; device rcl:C-EUC0805 -> rcl:C-EUC0402
- C39: value 1uF -> 10uF; device rcl:C-EUC0402 -> rcl:C-EUC0805
- C8: value 10uF -> 1uF; device rcl:C-EUC0805 -> rcl:C-EUC0402
- CN2: value TSW-120-08-L-S-RA -> 48204-0001; device m0wut:CONN_0.1"_1X20 -> m0wut:USB_4WAY""
- CN3: value 48204-0001 -> (none); device m0wut:USB_4WAY"" -> m0wut:USBWURTH
- CN4: value 1-1734530-1 -> TSW-120-08-L-S-RA; device m0wut:CONN_TE_DB-HD15 -> m0wut:CONN_0.1"_1X20
- CN5: value (none) -> 1-1734530-1; device m0wut:USBWURTH -> m0wut:CONN_TE_DB-HD15
- IC1: value FT230XQ -> TUSB2046BIRHBT; device ftdichip:FT230XQ -> texas:TUSB2046BIRHBIRHB
- IC2: value TUSB2046BIRHBT -> FT230XQ; device texas:TUSB2046BIRHBIRHB -> ftdichip:FT230XQ
- IC3: value IC_MAX3313 -> FT230XQ; device m0wut:IC_MAX3313 -> ftdichip:FT230XQ
- IC5: value FT230XQ -> (none); device ftdichip:FT230XQ -> m0wut:MCP1700
- IC6: value (none) -> IC_MAX3313; device m0wut:MCP1700 -> m0wut:IC_MAX3313
- L1: value (none) -> 100uH
- L4: value 100uH -> (none)
- R1, R2: value 1k5 -> 27
- R10: value 100k -> 27
- R12: value (none) -> 27
- R14: value 27 -> 1k5
- R15: value (none) -> 10k
- R16: value (none) -> 69k8
- R17: value 220 -> 100k
- R18: value 220 -> 2k2
- R23: value 220 -> 0R
- R29: value 137k -> 220
- R3: value 0R -> 27
- R30, R31: value (none) -> 220
- R32: value (none) -> 137k
- R4: value 15k -> 27
- R7: value (none) -> 15k
- R8: value (none) -> 1k5
- R9: value 69k8 -> 27
- RN1: value 2k2 -> 27
- RN3: value 27 -> 2k2
- renumbered R33 to R12, U$1 to CN6
Connections:
- net !MCLR: now also C17.1, R15.1; no longer C3.1, R35.1
- net +3V3: now also C13.1, C14.1, C15.1, C2.1, C3.1, C34.1, C39.1, C6.1, C7.1, IC1.!EXTMEM, IC1.!OVRCUR1, IC1.!OVRCUR2, IC1.!OVRCUR3, IC1.!OVRCUR4, IC1.VCC@1, IC2.!RESET, IC2.3V3OUT, IC2.VCCIO, IC3.!RESET, IC3.3V3OUT, IC3.VCC, IC3.VCCIO, IC5.VO, R14.2, R15.2, R7.1, R8.2; no longer C10.1, C11.1, C25.1, C29.1, C30.1, C40.1, C41.1, C8.1, C9.1, IC1.!RESET, IC1.3V3OUT, IC1.VCCIO, IC2.!EXTMEM, IC2.!OVRCUR1, IC2.!OVRCUR2, IC2.!OVRCUR3, IC2.!OVRCUR4, IC2.VCC@1, IC5.!RESET, IC5.3V3OUT, IC5.VCC, IC5.VCCIO, IC6.VO, R1.2, R2.2, R35.2, R4.1
- net +5V: now also C18.1, C19.1, C4.1, C5.1, CN2.VBUS, IC5.VI, L1.2, L4.1, R16.2, R18.2, RN3.1, RN3.2, RN3.3; no longer C31.1, C32.1, C34.1, C38.1, CN5.VBUS, IC6.VI, L4.2, L6.1, R34.2, R9.2, RN1.1, RN1.2, RN1.3
- net 232_DTR: now also CN4.P$2; no longer CN2.P$2
- net 232_FROM_P3: now also L6.2; no longer L5.2
- net 232_RTS: now also CN4.P$4; no longer CN2.P$4
- net 232_RXD: now also C38.1, CN4.P$5, L3.2; no longer C28.1, CN2.P$5, L2.2
- net 232_TO_P3: now also L5.2; no longer L1.2
- net 232_TXD: now also C37.1, CN4.P$3, L2.2; no longer C27.1, CN2.P$3, L3.2
- net 5V_IN: now also C35.1, CN4.P$20, L1.1; no longer C26.1, CN2.P$20, L4.1
- net ACC_ALC: now also CN4.P$12, R16.1, R17.2, R32.1; no longer CN2.P$12, R10.2, R29.1, R9.1
- net ACC_AUX: now also CN4.P$15, R20.1; no longer CN2.P$15, R18.1
- net ACC_BND0: now also CN4.P$7, R30.1, RN3.1A; no longer CN2.P$7, R27.1, RN1.1A
- net ACC_BND1: now also CN4.P$14, R18.1, R21.1; no longer CN2.P$14, R19.1, R34.1
- net ACC_BND2: now also CN4.P$9, R27.1, RN3.3A; no longer CN2.P$9, R24.1, RN1.3A
- net ACC_BND3: now also CN4.P$8, R31.1, RN3.2A; no longer CN2.P$8, R28.1, RN1.2A
- net ACC_COMMON: now also C20.1, CN5.12, CN5.5, R23.2; no longer C33.1, CN4.12, CN4.5, R3.2
- net ACC_DI0: now also CN4.P$16, R19.1; no longer CN2.P$16, R17.1
- net ACC_DI1: now also CN4.P$17, R25.1; no longer CN2.P$17, R22.1
- net ACC_DO0: now also CN4.P$18, R24.1; no longer CN2.P$18, R21.1
- net ACC_DO1: now also CN4.P$19, R29.1; no longer CN2.P$19, R26.1
- net ACC_KEY: now also CN4.P$10, R28.1; no longer CN2.P$10, R25.1
- net ACC_PTT: now also CN4.P$13, R22.1; no longer CN2.P$13, R20.1
- net ACC_PWR: now also CN4.P$11, R26.1; no longer CN2.P$11, R23.1
- net AGND: now also C25.2, C26.2, C29.2, C30.2, C31.2, C32.2, C37.2, C38.2, CN5.TAB; no longer C12.2, C13.2, C14.2, C15.2, C16.2, C17.2, C18.2, C19.2, CN4.TAB
- net ALC_X: now also C33.1, CN5.15, R32.2; no longer C24.1, CN4.15, R29.2
- net ASDF: now also L2.1; no longer L3.1
- net AUX_X: now also C22.1, CN5.2, R20.2; no longer C13.1, CN4.2, R18.2
- net BND0_X: now also C31.1, CN5.13, R30.2; no longer C22.1, CN4.13, R27.2
- net BND1_X: now also C23.1, CN5.3, R21.2; no longer C14.1, CN4.3, R19.2
- net BND2_X: now also C28.1, CN5.9, R27.2; no longer C19.1, CN4.9, R24.2
- net BND3_X: now also C32.1, CN5.14, R31.2; no longer C23.1, CN4.14, R28.2
- net D+_P: now also R1.1; no longer R11.1
- net DIG0_X: now also C21.1, CN5.1, R19.2; no longer C12.1, CN4.1, R17.2
- net DIG1_X: now also C26.1, CN5.7, R25.2; no longer C17.1, CN4.7, R22.2
- net DIGO1_X: now also C30.1, CN5.11, R29.2; no longer C21.1, CN4.11, R26.2
- net DIGO_X: now also C25.1, CN5.6, R24.2; no longer C16.1, CN4.6, R21.2
- net DM0: now also IC1.DM0, R2.2; no longer IC2.DM0, R14.2
- net DM1: now also CN2.D-, R3.1, RN1.1A; no longer CN3.D-, R7.1, RN2.1A
- net DM2: now also CN3.D-, R5.1, RN1.3A; no longer CN5.D-, R15.1, RN2.3A
- net DM3: now also IC3.USBDM, RN2.1A; no longer IC5.USBDM, RN3.1A
- net DM4: now also IC2.USBDM, R10.2, RN2.3A; no longer IC1.USBDM, R31.2, RN3.3A
- net DP0: now also IC1.DP0, R1.2, R8.1; no longer IC2.DP0, R11.2, R13.1
- net DP1: now also CN2.D+, R4.1, RN1.2A; no longer CN3.D+, R8.1, RN2.2A
- net DP2: now also CN3.D+, R6.1, RN1.4A; no longer CN5.D+, R16.1, RN2.4A
- net DP3: now also IC3.USBDP, R11.2, R14.1, RN2.2A; no longer IC5.USBDP, R2.1, R32.2, RN3.2A
- net DP4: now also IC2.USBDP, R13.1, R9.2, RN2.4A; no longer IC1.USBDP, R1.1, R30.2, RN3.4A
- net GND: now also C12.2, C13.2, C14.2, C15.2, C16.2, C17.2, C18.2, C19.2, C35.2, CN2.GND, CN2.SHIELD, CN3.ID, CN4.P$1, CN4.P$6, IC1.BUSPWR, IC1.EEDATA/GANGED, IC1.PAD, IC1.TSTMODE, IC1.TSTPLL/48MCLK, IC3.GND@1, R17.1, R23.1, RN1.1, RN1.2, RN1.3, RN1.4; no longer C25.2, C26.2, C29.2, C30.2, C31.2, C32.2, C37.2, C38.2, C41.2, CN2.P$1, CN2.P$6, CN5.GND, CN5.ID, CN5.SHIELD, IC2.BUSPWR, IC2.EEDATA/GANGED, IC2.PAD, IC2.TSTMODE, IC2.TSTPLL/48MCLK, IC5.GND@1, R10.1, R3.1, RN3.1, RN3.2, RN3.3, RN3.4
- net KEY_X: now also C29.1, CN5.10, R28.2; no longer C20.1, CN4.10, R25.2
- net N$1: now also IC1.DM4, R10.1; no longer IC2.DM4, R31.1
- net N$10: now also IC1.XTAL2; no longer IC2.XTAL2
- net N$11: now also IC1.DM2, R5.2; no longer IC2.DM2, R15.2
- net N$12: now also IC1.DM1, R3.2; no longer IC2.DM1, R7.2
- net N$13: now also IC1.DP1, R4.2; no longer IC2.DP1, R8.2
- net N$14: now also IC1.DP2, R6.2; no longer IC2.DP2, R16.2
- net N$15: now also C42.1, IC6.V-; no longer C37.1, IC3.V-
- net N$16: now also IC1.DP3, R11.1; no longer IC2.DP3, R32.1
- net N$17: now also IC1.DM3; no longer IC2.DM3
- net N$2: now also C16.1; no longer C2.1
- net N$20: now also R2.1; no longer R14.1
- net N$3: now also IC1.DP4, R9.1; no longer IC2.DP4, R30.1
- net N$4: now also C40.1, IC6.VCC, L4.2; no longer C42.1, IC3.VCC, L6.2
- net N$6: now also C41.1, IC6.C1-; no longer C35.1, IC3.C1-
- net N$7: now also C41.2, IC6.C1+; no longer C35.2, IC3.C1+
- net N$8: now also IC1.XTAL1; no longer IC2.XTAL1
- net N$9: now also C8.1, IC1.!RESET, R7.2; no longer C39.1, IC2.!RESET, R4.2
- net PTT_X: now also C24.1, CN5.4, R22.2; no longer C15.1, CN4.4, R20.2
- net PWR_X: now also C27.1, CN5.8, R26.2; no longer C18.1, CN4.8, R23.2
- net SADF: now also L3.1; no longer L2.1
- net UART_FROM_CAT: now also C9.1, IC2.RXD; no longer C5.1, IC1.RXD
- net UART_FROM_P3: now also IC6.ROUT; no longer IC3.ROUT
- net UART_FROM_WK: now also C11.1, IC3.RXD; no longer C7.1, IC5.RXD
- net UART_TO_CAT: now also C12.1, IC2.TXD; no longer C4.1, IC1.TXD
- net UART_TO_P3: now also IC6.TIN; no longer IC3.TIN
- net UART_TO_WK: now also C10.1, IC3.TXD; no longer C6.1, IC5.TXD
- net WTRE: now also IC6.TOUT, L5.1; no longer IC3.TOUT, L1.1
- net Y5W4: now also IC6.RIN, L6.1; no longer IC3.RIN, L5.1

Commit message: minor code fixes
Parts:
- L4: value (none) -> 100uH
- RN1, RN2: value 27 -> 15k
Changed lines of the file:
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@@
 <part name="GND13" library="supply1" deviceset="GND" device=""/>
 <part name="GND14" library="supply1" deviceset="GND" device=""/>
-<part name="RN2" library="m0wut" deviceset="R_BOURNS_CAY16-J4" device="" value="27"/>
+<part name="RN2" library="m0wut" deviceset="R_BOURNS_CAY16-J4" device="" value="15k"/>
 <part name="C6" library="rcl" deviceset="C-EU" device="C0402" value="100nF"/>
 <part name="C7" library="rcl" deviceset="C-EU" device="C0402" value="100nF"/>
@@
 <part name="R11" library="rcl" deviceset="R-EU_" device="R0402" value="27"/>
 <part name="R12" library="rcl" deviceset="R-EU_" device="R0402" value="27"/>
-<part name="RN1" library="m0wut" deviceset="R_BOURNS_CAY16-J4" device="" value="27"/>
+<part name="RN1" library="m0wut" deviceset="R_BOURNS_CAY16-J4" device="" value="15k"/>
 <part name="GND8" library="supply1" deviceset="GND" device=""/>
 <part name="Q1" library="adafruit" deviceset="MOSFET-N" device="REFLOW"/>
@@
 <part name="SUPPLY6" library="supply2" deviceset="AGND" device=""/>
 <part name="SUPPLY7" library="supply2" deviceset="AGND" device=""/>
-<part name="L4" library="m0wut" deviceset="INDUCTOR" device=""/>
+<part name="L4" library="m0wut" deviceset="INDUCTOR" device="" value="100uH"/>
 </parts>
 <sheets>
