File: KIO_WUT.kicad_pcb (KiCad board)
At the start: 4 copper layers, 77.4 x 32.6 mm, 85 parts, among them J1 TSW-120-08-T-S-RA, J2 USB_C_Receptacle, J3 AudioJack3_SwitchTR, J4 DB15_Female_HighDensity_Mount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, Q1 SI1539CDL-T1-GE3, Q2 FDC6303N, Q3 FDC6303N, U1 TCMT1600, U2 TCMT1600, U3 TCMT1600, U4 TCMT1600, U5 93LC56BT-E/OT, U6 FT2232HQ, U7 WK3IC, Y1 ABM10AIG-12.000MHZ-7-D2Z-T

Commit message: .
Parts:
- removed D2, D3: KPT-1608SURCK, LED_SMD:LED_0603_1608Metric
- removed R17, R18: 1k, Resistor_SMD:R_0402_1005Metric
- C1, C10, C11, C12, C13, C14, C16, C2, C3, C4, C5, C6, C7, C8, C9, D1, D4, D5, FL1, H1, L1, Q1, R1, R12, R13, R16, R2, R5, R6, R9, RN1, RN2, RN3, U1, U2, U3, U4, U5, U6, U7: moved to F.Cu
- J1, J2, J3, J4: moved to B.Cu
- moved FB1 116.8 mm to (99.0, 99.8), turned to 90 degrees
- moved FB2 111.0 mm to (102.2, 99.8), turned to 90 degrees
- moved L1 72.6 mm to (63.9, 96.2)
- moved C11 62.6 mm to (68.9, 104.5)
- moved C2 62.6 mm to (68.9, 102.0)
- moved RN3 62.6 mm to (68.9, 96.7)
- moved C4 61.6 mm to (69.4, 99.5)
- moved D4 60.5 mm to (130.5, 102.7), turned to 180 degrees
- moved D5 59.8 mm to (130.5, 97.2), turned to 180 degrees
- moved C3 56.6 mm to (71.9, 97.0)
- moved U7 54.3 mm to (127.2, 86.8), turned to 90 degrees
- moved J3 53.9 mm to (127.2, 107.5), turned to 0 degrees
- moved C5 53.1 mm to (73.7, 97.2), turned to 180 degrees
- moved C17 51.4 mm to (108.0, 99.5), turned to 90 degrees
- moved C31 49.9 mm to (122.5, 93.0), turned to -90 degrees
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Connections:
- Q2 pad 4: ~PTT -> /CAT and Winkey/~PTT
- Q2 pad 6: ~PTT -> /CAT and Winkey/~PTT
- Q3 pad 4: ~KEY -> /CAT and Winkey/~KEY
- Q3 pad 6: ~KEY -> /CAT and Winkey/~KEY
- R7 pad 1: /~KEY -> /CAT and Winkey/~PTT
- R8 pad 1: /~PTT -> /CAT and Winkey/~KEY
- U6 pad 29: Net-(R18-Pad1) -> unconnected-(U6-Pad29)
- U6 pad 30: Net-(R18-Pad1) -> unconnected-(U6-Pad30)
- U6 pad 54: Net-(R17-Pad2) -> unconnected-(U6-Pad54)
- U6 pad 55: Net-(R17-Pad2) -> unconnected-(U6-Pad55)
Routing:
- net GNDA: track 19.0 -> 0.00 mm
- net /ACC_PWR: track 2.14 -> 12.3 mm
- net /CAT and Winkey/CW_DOT: track 11.3 -> 3.64 mm
- net /D_P: track 4.74 -> 11.0 mm
- net /D_N: track 4.74 -> 10.3 mm
- net /CAT and Winkey/CW_DASH: track 6.16 -> 0.78 mm
- net /RS232_RXD: track 4.47 -> 0.00 mm
- net Net-(R13-Pad1): track 4.35 -> 0.00 mm
- net GND: track 14.5 -> 10.4 mm
- net Net-(C21-Pad1): track 0.00 -> 3.78 mm
- net Net-(C19-Pad1): track 0.00 -> 3.65 mm
- net /RS232_DTR: track 3.11 -> 0.00 mm
- net Net-(C1-Pad1): track 3.05 -> 0.00 mm, vias 2 -> 0
- net /ACC_COM: track 44.6 -> 47.5 mm
- net /CAT and Winkey/1V8: track 0.00 -> 2.92 mm
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- added copper zone on In1.Cu, net GND
- added copper zone on B.Cu, net GNDPWR
- removed copper zone on In2.Cu, net GND
- removed copper zone on F.Cu, net GNDPWR
