File: _autosave-ft2232.kicad_sch (KiCad schematic)
At the start: 41 parts, among them Q1 SI1539CDL-T1-GE3, Q2 FDC6303N, Q3 FDC6303N, U5 93LC56BT-E/OT, U6 FT2232HQ, U7 WK3IC, Y1 ABM10AIG-12.000MHZ-7-D2Z-T

Commit message: .
Parts:
- removed D2, D3: KPT-1608SURCK, LED_SMD:LED_0603_1608Metric, symbol Device:LED
- removed R17, R18: 1k, Resistor_SMD:R_0402_1005Metric, symbol Device:R
Connections:
- net at U6.29 (ACBUS3): no longer U6.30 (ACBUS4)
- net at U6.54 (BCBUS3): no longer U6.55 (BCBUS4)
- no-connect marks 32 -> 36
Changed lines of the file:
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@@
   (junction (at 139.7 40.64) (diameter 1.016) (color 0 0 0 0))
   (junction (at 139.7 52.07) (diameter 1.016) (color 0 0 0 0))
-  (junction (at 142.24 92.71) (diameter 1.016) (color 0 0 0 0))
-  (junction (at 142.24 138.43) (diameter 1.016) (color 0 0 0 0))
   (junction (at 146.05 33.02) (diameter 1.016) (color 0 0 0 0))
   (junction (at 146.05 52.07) (diameter 1.016) (color 0 0 0 0))
@@
   (no_connect (at 138.43 87.63))
   (no_connect (at 138.43 90.17))
+  (no_connect (at 138.43 92.71))
+  (no_connect (at 138.43 95.25))
   (no_connect (at 138.43 97.79))
   (no_connect (at 138.43 100.33))
@@
   (no_connect (at 138.43 133.35))
   (no_connect (at 138.43 135.89))
+  (no_connect (at 138.43 138.43))
+  (no_connect (at 138.43 140.97))
   (no_connect (at 138.43 143.51))
   (no_connect (at 138.43 146.05))
@@
     (stroke (width 0) (type solid) (color 0 0 0 0))
   )
-  (wire (pts (xy 138.43 92.71) (xy 142.24 92.71))
-    (stroke (width 0) (type solid) (color 0 0 0 0))
-  )
-  (wire (pts (xy 138.43 95.25) (xy 142.24 95.25))
-    (stroke (width 0) (type solid) (color 0 0 0 0))
-  )
   (wire (pts (xy 138.43 107.95) (xy 165.1 107.95))
     (stroke (width 0) (type solid) (color 0 0 0 0))
@@
     (stroke (width 0) (type solid) (color 0 0 0 0))
   )
-  (wire (pts (xy 138.43 138.43) (xy 142.24 138.43))
-    (stroke (width 0) (type solid) (color 0 0 0 0))
-  )
-  (wire (pts (xy 138.43 140.97) (xy 142.24 140.97))
-    (stroke (width 0) (type solid) (color 0 0 0 0))
-  )
   (wire (pts (xy 139.7 21.59) (xy 128.27 21.59))
     (stroke (width 0) (type solid) (color 0 0 0 0))
@@
     (stroke (width 0) (type solid) (color 0 0 0 0))
   )
-  (wire (pts (xy 142.24 92.71) (xy 148.59 92.71))
-    (stroke (width 0) (type solid) (color 0 0 0 0))
-  )
-  (wire (pts (xy 142.24 95.25) (xy 142.24 92.71))
-    (stroke (width 0) (type solid) (color 0 0 0 0))
-  )
-  (wire (pts (xy 142.24 138.43) (xy 142.24 140.97))
-    (stroke (width 0) (type solid) (color 0 0 0 0))
-  )
-  (wire (pts (xy 142.24 138.43) (xy 146.05 138.43))
-    (stroke (width 0) (type solid) (color 0 0 0 0))
-  )
   (wire (pts (xy 143.51 67.31) (xy 138.43 67.31))
     (stroke (width 0) (type solid) (color 0 0 0 0))
@@
     (stroke (width 0) (type solid) (color 0 0 0 0))
   )
-  (wire (pts (xy 146.05 119.38) (xy 146.05 118.11))
-    (stroke (width 0) (type solid) (color 0 0 0 0))
-  )
-  (wire (pts (xy 146.05 127) (xy 146.05 128.27))
-    (stroke (width 0) (type solid) (color 0 0 0 0))
-  )
-  (wire (pts (xy 146.05 135.89) (xy 146.05 138.43))
-    (stroke (width 0) (type solid) (color 0 0 0 0))
-  )
   (wire (pts (xy 151.13 21.59) (xy 151.13 24.13))
     (stroke (width 0) (type solid) (color 0 0 0 0))
@@
     (stroke (width 0) (type solid) (color 0 0 0 0))
   )
-  (wire (pts (xy 156.21 92.71) (xy 163.83 92.71))
-    (stroke (width 0) (type solid) (color 0 0 0 0))
-  )
   (wire (pts (xy 161.29 68.58) (xy 143.51 68.58))
     (stroke (width 0) (type solid) (color 0 0 0 0))
@@
   )
   (wire (pts (xy 162.56 52.07) (xy 162.56 50.8))
-    (stroke (width 0) (type solid) (color 0 0 0 0))
-  )
-  (wire (pts (xy 163.83 78.74) (xy 163.83 80.01))
-    (stroke (width 0) (type solid) (color 0 0 0 0))
-  )
-  (wire (pts (xy 163.83 87.63) (xy 163.83 92.71))
     (stroke (width 0) (type solid) (color 0 0 0 0))
   )
@@
     )
     (property "Datasheet" "" (id 3) (at 55.88 97.79 0)
-      (effects (font (size 1.27 1.27)) hide)
-    )
-    (pin "1")
-  )
-  (symbol (lib_id "power:+3.3V") (at 146.05 118.11 0) (unit 1)
-    (in_bom yes) (on_board yes)
-    (property "Reference" "#PWR043" (id 0) (at 146.05 121.92 0)
-      (effects (font (size 1.27 1.27)) hide)
-    )
-    (property "Value" "+3.3V" (id 1) (at 147.32 113.03 0))
-    (property "Footprint" "" (id 2) (at 146.05 118.11 0)
-      (effects (font (size 1.27 1.27)) hide)
-    )
-    (property "Datasheet" "" (id 3) (at 146.05 118.11 0)
-      (effects (font (size 1.27 1.27)) hide)
-    )
-    (pin "1")
-  )
-  (symbol (lib_id "power:+3.3V") (at 163.83 78.74 0) (unit 1)
-    (in_bom yes) (on_board yes)
-    (property "Reference" "#PWR044" (id 0) (at 163.83 82.55 0)
-      (effects (font (size 1.27 1.27)) hide)
-    )
-    (property "Value" "+3.3V" (id 1) (at 164.1983 74.4156 0))
-    (property "Footprint" "" (id 2) (at 163.83 78.74 0)
-      (effects (font (size 1.27 1.27)) hide)
-    )
-    (property "Datasheet" "" (id 3) (at 163.83 78.74 0)
       (effects (font (size 1.27 1.27)) hide)
     )
@@
     (pin "2")
   )
-  (symbol (lib_id "Device:R") (at 146.05 132.08 0) (unit 1)
-    (in_bom yes) (on_board yes)
-    (property "Reference" "R17" (id 0) (at 147.8281 130.9306 0)
-      (effects (font (size 1.27 1.27)) (justify left))
-    )
-    (property "Value" "1k" (id 1) (at 147.828 133.229 0)
-      (effects (font (size 1.27 1.27)) (justify left))
-    )
-    (property "Footprint" "Resistor_SMD:R_0402_1005Metric" (id 2) (at 144.272 132.08 90)
-      (effects (font (size 1.27 1.27)) hide)
-    )
-    (property "Datasheet" "~" (id 3) (at 146.05 132.08 0)
-      (effects (font (size 1.27 1.27)) hide)
-    )
-    (pin "1")
-    (pin "2")
-  )
-  (symbol (lib_id "Device:R") (at 152.4 92.71 90) (unit 1)
-    (in_bom yes) (on_board yes)
-    (property "Reference" "R18" (id 0) (at 152.4 87.4838 90))
-    (property "Value" "1k" (id 1) (at 152.4 89.783 90))
-    (property "Footprint" "Resistor_SMD:R_0402_1005Metric" (id 2) (at 152.4 94.488 90)
-      (effects (font (size 1.27 1.27)) hide)
-    )
-    (property "Datasheet" "~" (id 3) (at 152.4 92.71 0)
-      (effects (font (size 1.27 1.27)) hide)
-    )
-    (pin "1")
-    (pin "2")
-  )
   (symbol (lib_id "Device:R") (at 177.8 101.6 0) (unit 1)
     (in_bom yes) (on_board yes)
@@
       (effects (font (size 1.27 1.27)) hide)
     )
-    (pin "1")
-    (pin "2")
-  )
-  (symbol (lib_id "Device:LED") (at 146.05 123.19 90) (unit 1)
-    (in_bom yes) (on_board yes)
-    (property "Reference" "D2" (id 0) (at 149.86 123.19 90)
-      (effects (font (size 1.27 1.27)) (justify right))
-    )
-    (property "Value" "KPT-1608SURCK " (id 1) (at 149.86 125.73 90)
-      (effects (font (size 1.27 1.27)) (justify right))
-    )
-    (property "Footprint" "LED_SMD:LED_0603_1608Metric" (id 2) (at 146.05 123.19 0)
-      (effects (font (size 1.27 1.27)) hide)
-    )
-    (property "Datasheet" "~" (id 3) (at 146.05 123.19 0)
-      (effects (font (size 1.27 1.27)) hide)
-    )
-    (pin "1")
-    (pin "2")
-  )
-  (symbol (lib_id "Device:LED") (at 163.83 83.82 90) (unit 1)
-    (in_bom yes) (on_board yes)
-    (property "Reference" "D3" (id 0) (at 167.64 83.82 90)
-      (effects (font (size 1.27 1.27)) (justify right))
-    )
-    (property "Value" "KPT-1608SURCK " (id 1) (at 167.64 86.36 90)
-      (effects (font (size 1.27 1.27)) (justify right))
-    )
-    (property "Footprint" "LED_SMD:LED_0603_1608Metric" (id 2) (at 163.83 83.82 0)
-      (effects (font (size 1.27 1.27)) hide)
-    )
-    (property "Datasheet" "~" (id 3) (at 163.83 83.82 0)
-      (effects (font (size 1.27 1.27)) hide)
-    )
