File: KIO_WUT.kicad_sch (KiCad schematic)
At the start: 44 parts, among them J1 TSW-120-08-T-S-RA, J2 USB_C_Receptacle, J3 AudioJack3_SwitchTR, J4 DB15_Female_HighDensity_Mount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, U1 TCMT1600, U2 TCMT1600, U3 TCMT1600, U4 TCMT1600

Commit message: .
Connections:
- net CAT and Winkey/~KEY: now also R8.1; no longer R7.1
- net CAT and Winkey/~PTT: now also R7.1; no longer R8.1
Changed lines of the file:
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@@
-(kicad_sch (version 20210406) (generator eeschema)
+(kicad_sch (version 20210606) (generator eeschema)
   (paper "A3")
   (junction (at 63.5 71.12) (diameter 0.9144) (color 0 0 0 0))
@@
       (effects (font (size 1.27 1.27)) hide)
     )
-    (property "Datasheet" " ~" (id 3) (at 318.77 184.15 0)
+    (property "Datasheet" " ~{}" (id 3) (at 318.77 184.15 0)
       (effects (font (size 1.27 1.27)) hide)
     )
@@
       (effects (font (size 1.27 1.27)) (justify left top))
     )
-    (pin "~KEY" output (at 302.26 110.49 0)
-      (effects (font (size 1.27 1.27)) (justify right))
-    )
     (pin "UART_PC_TO_CAT" output (at 302.26 123.19 0)
       (effects (font (size 1.27 1.27)) (justify right))
@@
       (effects (font (size 1.27 1.27)) (justify left))
     )
-    (pin "~PTT" output (at 302.26 113.03 0)
+    (pin "USB_N" bidirectional (at 264.16 120.65 180)
+      (effects (font (size 1.27 1.27)) (justify left))
+    )
+    (pin "USB_P" bidirectional (at 264.16 118.11 180)
+      (effects (font (size 1.27 1.27)) (justify left))
+    )
+    (pin "~PTT" output (at 302.26 110.49 0)
       (effects (font (size 1.27 1.27)) (justify right))
     )
-    (pin "USB_N" bidirectional (at 264.16 120.65 180)
-      (effects (font (size 1.27 1.27)) (justify left))
-    )
-    (pin "USB_P" bidirectional (at 264.16 118.11 180)
-      (effects (font (size 1.27 1.27)) (justify left))
-    )
-  )
+    (pin "~KEY" output (at 302.26 113.03 0)
+      (effects (font (size 1.27 1.27)) (justify right))
+    )
+  )
